File: eagle/wifi-test-middle.brd (EAGLE design)
At the start: 50.8 x 68.6 mm, 18 parts

Commit message: updated middle board hole size
Parts:
- E$1, E$2: device Pinoccio:1X16_2MM_POGO-HOLES -> Pinoccio:1X16_2MM_POGO-HOLES-06
- E$11, E$12, E$13, E$14, E$15, E$16, E$3, E$4, E$5, E$6, E$7, E$8: device Pinoccio:1X1_2MM_POGO-HOLES -> Pinoccio:1X1_2MM_POGO-HOLES_055
Other:
- board text added: "Pinoccio(tm) Wi-Fi Test Jig - Middle v1.1"
- board text removed: "Pinoccio(tm) Wi-Fi Test Jig - Middle v1.0"
Changed lines of the file:
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@@
 <text x="-10.4394" y="-8.3312" size="1.27" layer="51" font="vector" ratio="15">http://pinocc.io</text>
 <text x="-10.414" y="-6.604" size="1.27" layer="51" font="vector" ratio="15">Design by: Eric Jennings for Pinoccio</text>
-<text x="-10.3632" y="-4.8514" size="1.778" layer="51" font="vector" ratio="15">Pinoccio(tm) Wi-Fi Test Jig - Middle v1.0</text>
+<text x="-10.3632" y="-4.8514" size="1.778" layer="51" font="vector" ratio="15">Pinoccio(tm) Wi-Fi Test Jig - Middle v1.1</text>
 <text x="-10.4648" y="-10.2362" size="1.27" layer="51" font="vector" ratio="15">Licensed under CERN OHL v.1.1</text>
 <text x="48.1584" y="49.9364" size="1.016" layer="21" font="vector" ratio="15">GS1011</text>
@@
 <element name="JP9" library="Pinoccio" package="STAND-OFF" value="STAND-OFF" x="33.02" y="9.3726" locked="yes"/>
 <element name="JP10" library="Pinoccio" package="STAND-OFF" value="STAND-OFF" x="68.58" y="9.3726" locked="yes"/>
-<element name="E$1" library="Pinoccio" package="1X16_2MM_POGO-HOLES" value="" x="39.751" y="39.37" rot="R270"/>
-<element name="E$2" library="Pinoccio" package="1X16_2MM_POGO-HOLES" value="" x="61.849" y="39.37" rot="R270"/>
-<element name="E$3" library="Pinoccio" package="1X1_2MM_POGO-HOLES" value="" x="48.26" y="39.878"/>
-<element name="E$4" library="Pinoccio" package="1X1_2MM_POGO-HOLES" value="" x="50.8" y="39.878"/>
-<element name="E$5" library="Pinoccio" package="1X1_2MM_POGO-HOLES" value="" x="53.34" y="39.878"/>
-<element name="E$6" library="Pinoccio" package="1X1_2MM_POGO-HOLES" value="" x="53.34" y="37.338"/>
-<element name="E$7" library="Pinoccio" package="1X1_2MM_POGO-HOLES" value="" x="50.8" y="37.338"/>
-<element name="E$8" library="Pinoccio" package="1X1_2MM_POGO-HOLES" value="" x="48.26" y="37.338"/>
-<element name="E$11" library="Pinoccio" package="1X1_2MM_POGO-HOLES" value="" x="48.26" y="48.0568"/>
-<element name="E$12" library="Pinoccio" package="1X1_2MM_POGO-HOLES" value="" x="50.8" y="48.0568"/>
-<element name="E$13" library="Pinoccio" package="1X1_2MM_POGO-HOLES" value="" x="53.34" y="48.0568"/>
-<element name="E$14" library="Pinoccio" package="1X1_2MM_POGO-HOLES" value="" x="53.34" y="45.5168"/>
-<element name="E$15" library="Pinoccio" package="1X1_2MM_POGO-HOLES" value="" x="50.8" y="45.5168"/>
-<element name="E$16" library="Pinoccio" package="1X1_2MM_POGO-HOLES" value="" x="48.26" y="45.5168"/>
+<element name="E$1" library="Pinoccio" package="1X16_2MM_POGO-HOLES-06" value="" x="39.751" y="39.37" rot="R270"/>
+<element name="E$2" library="Pinoccio" package="1X16_2MM_POGO-HOLES-06" value="" x="61.849" y="39.37" rot="R270"/>
+<element name="E$3" library="Pinoccio" package="1X1_2MM_POGO-HOLES_055" value="" x="48.26" y="39.878"/>
+<element name="E$4" library="Pinoccio" package="1X1_2MM_POGO-HOLES_055" value="" x="50.8" y="39.878"/>
+<element name="E$5" library="Pinoccio" package="1X1_2MM_POGO-HOLES_055" value="" x="53.34" y="39.878"/>
+<element name="E$6" library="Pinoccio" package="1X1_2MM_POGO-HOLES_055" value="" x="53.34" y="37.338"/>
+<element name="E$7" library="Pinoccio" package="1X1_2MM_POGO-HOLES_055" value="" x="50.8" y="37.338"/>
+<element name="E$8" library="Pinoccio" package="1X1_2MM_POGO-HOLES_055" value="" x="48.26" y="37.338"/>
+<element name="E$11" library="Pinoccio" package="1X1_2MM_POGO-HOLES_055" value="" x="48.26" y="48.0568"/>
+<element name="E$12" library="Pinoccio" package="1X1_2MM_POGO-HOLES_055" value="" x="50.8" y="48.0568"/>
+<element name="E$13" library="Pinoccio" package="1X1_2MM_POGO-HOLES_055" value="" x="53.34" y="48.0568"/>
+<element name="E$14" library="Pinoccio" package="1X1_2MM_POGO-HOLES_055" value="" x="53.34" y="45.5168"/>
+<element name="E$15" library="Pinoccio" package="1X1_2MM_POGO-HOLES_055" value="" x="50.8" y="45.5168"/>
+<element name="E$16" library="Pinoccio" package="1X1_2MM_POGO-HOLES_055" value="" x="48.26" y="45.5168"/>
 </elements>
 <signals>
